Commit message: added arm prefix xacro property

File: human_arm_description/urdf/hand.xacro (robot description, xacro)
@@ -1,5 +1,6 @@
 <?xml version='1.0'?>
 <robot name="hand" xmlns:xacro="http://www.ros.org/wiki/xacro">
-<link name="shoulder">
+<xacro:property name="prefix" value="right_"/>
+<link name="${prefix}shoulder">
     <inertial>
       <origin xyz="0 0 0" rpy="0 0 0" />
@@ -24,13 +25,13 @@
 </link>
 <joint
-    name="shoulder_humerus" type="revolute">
+    name="${prefix}shoulder_humerus" type="revolute">
     <origin xyz="0 0 0.015" rpy="0 0 0" />
-    <parent link="shoulder" />
-    <child link="humerus" />
+    <parent link="${prefix}shoulder" />
+    <child link="${prefix}humerus" />
     <axis xyz="1 0 0" />
     <limit lower="-3.14" upper="0.345" effort="10000" velocity="0.5"/>
     <dynamics damping="5" friction="0.0"/>
 </joint>
-<link name="humerus">
+<link name="${prefix}humerus">
     <inertial>
       <origin xyz="0 0 0" rpy="0 0 0" />
@@ -55,13 +56,13 @@
 </link>
 <joint
-    name="humerus_elbow" type="revolute">
+    name="${prefix}humerus_elbow" type="revolute">
     <origin xyz="-0.001 -0.15 0.0147" rpy="0 0 0" />
-    <parent link="humerus" />
-    <child link="elbow" />
+    <parent link="${prefix}humerus" />
+    <child link="${prefix}elbow" />
     <axis xyz="0 1 0" />
     <limit lower="-3.142" upper="0" effort="10000" velocity="0.5"/>
     <dynamics damping="5" friction="0.0"/>
 </joint>
-<link name="elbow">
+<link name="${prefix}elbow">
     <inertial>
       <origin xyz="0.00116385 -0.0740893 -0.0073153" rpy="-1.21278e-13 1.94289e-16 -0.0115373" />
@@ -86,13 +87,13 @@
 </link>
 <joint
-    name="elbow_forearm" type="revolute">
+    name="${prefix}elbow_forearm" type="revolute">
     <origin xyz="0.01 -0.145 -0.015" rpy="0 0 0" />
-    <parent link="elbow" />
-    <child link="forearm" />
+    <parent link="${prefix}elbow" />
+    <child link="${prefix}forearm" />
     <axis xyz="0 0 1" />
     <limit lower="0" upper="2.4" effort="10000" velocity="0.5"/>
     <dynamics damping="5" friction="0.0"/>
 </joint>
-<link name="forearm">
+<link name="${prefix}forearm">
     <inertial>
       <origin xyz="0.00116385 -0.0740893 -0.0073153" rpy="-1.21278e-13 1.94289e-16 -0.0115373" />
@@ -117,13 +118,13 @@
 </link>
 <joint
-    name="forearm_wristy" type="revolute">
+    name="${prefix}forearm_wristy" type="revolute">
     <origin xyz="0.000 -0.185 0.015" rpy="0 0 0" />
-    <parent link="forearm" />
-    <child link="wristy" />
+    <parent link="${prefix}forearm" />
+    <child link="${prefix}wristy" />
     <axis xyz="0 1 0" />
     <limit lower="-3.142" upper="2" effort="10000" velocity="0.5"/>
     <dynamics damping="5" friction="0.0"/>
 </joint>
-<link name="wristy">
+<link name="${prefix}wristy">
     <inertial>
       <origin xyz="0 0 0" rpy="0 0 0" />
@@ -148,13 +149,13 @@
 </link>
 <joint
-    name="wristy_wristx" type="revolute">
+    name="${prefix}wristy_wristx" type="revolute">
     <origin xyz="0.000 -0.06 0.002" rpy="0 0 0" />
-    <parent link="wristy" />
-    <child link="wristx" />
+    <parent link="${prefix}wristy" />
+    <child link="${prefix}wristx" />
     <axis xyz="0 0 1" />
     <limit lower="-0.697" upper="0.697" effort="10000" velocity="0.5"/>
     <dynamics damping="5" friction="0.0"/>
 </joint>
-<link name="wristx">
+<link name="${prefix}wristx">
     <inertial>
       <origin xyz="0 0 0" rpy="0 0 0" />
@@ -179,44 +180,44 @@
 </link>
 <joint
-    name="wristx_wristz" type="revolute">
+    name="${prefix}wristx_wristz" type="revolute">
     <origin xyz="0.000 -0.035 0.000" rpy="0 0 0" />
-    <parent link="wristx" />
-    <child link="wristz" />
+    <parent link="${prefix}wristx" />
+    <child link="${prefix}wristz" />
+    <axis xyz="1 0 0" />
+    <limit lower="-1" upper="1.57" effort="10000" velocity="0.5"/>
+    <dynamics damping="5" friction="0.0"/>
+</joint>
+<link name="${prefix}wristz">
+    <inertial>
+      <origin xyz="0 0 0" rpy="0 0 0" />
+      <mass value="0.7" />
+          <inertia ixx="0.003" ixy="0" ixz="0" iyy="0.0030" iyz="0" izz="0.0035"/>
+    </inertial>
+    <visual>
+      <origin xyz="0 0 0" rpy="0 0 0" />
+      <geometry>
+        <mesh  filename="package://human_arm_description/meshes/wristz.stl" />
+      </geometry>
+      <material name="">
+        <color rgba="0.79216 0.81961 0.93333 1" />
+      </material>
+    </visual>
+    <collision>
+      <origin xyz="0 0 0" rpy="0 0 0" />
+      <geometry>
+          <mesh  filename="package://human_arm_description/meshes/wristz.stl" />
+      </geometry>
+    </collision>
+</link>
+<joint
+    name="${prefix}wristz_palm" type="fixed">
+    <origin xyz="0.03 -0.02 0.000" rpy="0 0 0" />
+    <parent link="${prefix}wristz" />
+    <child link="${prefix}palm" />
     <axis xyz="0 0 1" />
     <limit lower="-0.697" upper="1.57" effort="10000" velocity="0.5"/>
     <dynamics damping="5" friction="0.0"/>
 </joint>
-<link name="wristz">
-    <inertial>
-      <origin xyz="0 0 0" rpy="0 0 0" />
-      <mass value="0.7" />
-          <inertia ixx="0.003" ixy="0" ixz="0" iyy="0.0030" iyz="0" izz="0.0035"/>
-    </inertial>
-    <visual>
-      <origin xyz="0 0 0" rpy="0 0 0" />
-      <geometry>
-        <mesh  filename="package://human_arm_description/meshes/wristz.stl" />
-      </geometry>
-      <material name="">
-        <color rgba="0.79216 0.81961 0.93333 1" />
-      </material>
-    </visual>
-    <collision>
-      <origin xyz="0 0 0" rpy="0 0 0" />
-      <geometry>
-          <mesh  filename="package://human_arm_description/meshes/wristz.stl" />
-      </geometry>
-    </collision>
-</link>
-<joint
-    name="wristz_palm" type="fixed">
-    <origin xyz="0.03 -0.02 0.000" rpy="0 0 0" />
-    <parent link="wristz" />
-    <child link="palm" />
-    <axis xyz="0 0 1" />
-    <limit lower="-0.697" upper="1.57" effort="10000" velocity="0.5"/>
-    <dynamics damping="5" friction="0.0"/>
-</joint>
-<link name="palm">
+<link name="${prefix}palm">
     <inertial>
       <origin xyz="0 0 0" rpy="0 0 0" />
@@ -244,13 +245,13 @@
 ##################### INDEX FINGER ######################################## -->
 <joint
-    name="palm_index0" type="revolute">
+    name="${prefix}palm_index0" type="revolute">
     <origin xyz="0.010 -0.060 0.000" rpy="0 0 0" />
-    <parent link="palm" />
-    <child link="index0" />
-    <axis xyz="0 0 1" />
-    <limit lower="-0.697" upper="1.57" effort="10000" velocity="0.5"/>
-    <dynamics damping="5" friction="0.0"/>
-</joint>
-<link name="index0">
+    <parent link="${prefix}palm" />
+    <child link="${prefix}index0" />
+    <axis xyz="0 0 1" />
+    <limit lower="-0.3" upper="0.3" effort="10000" velocity="0.5"/>
+    <dynamics damping="5" friction="0.0"/>
+</joint>
+<link name="${prefix}index0">
     <inertial>
       <origin xyz="0 0 0" rpy="0 0 0" />
@@ -275,13 +276,13 @@
 </link>
 <joint
-    name="index0_index1" type="revolute">
+    name="${prefix}index0_index1" type="revolute">
     <origin xyz="0.00 -0.015 0.000" rpy="0 0 0" />
-    <parent link="index0" />
-    <child link="index1" />
-    <axis xyz="1 0 0" />
-    <limit lower="-0.697" upper="1.57" effort="10000" velocity="0.5"/>
-    <dynamics damping="5" friction="0.0"/>
-</joint>
-<link name="index1">
+    <parent link="${prefix}index0" />
+    <child link="${prefix}index1" />
+    <axis xyz="1 0 0" />
+    <limit lower="-0.2" upper="1.57" effort="10000" velocity="0.5"/>
+    <dynamics damping="5" friction="0.0"/>
+</joint>
+<link name="${prefix}index1">
     <inertial>
       <origin xyz="0 0 0" rpy="0 0 0" />
@@ -306,44 +307,44 @@
 </link>
 <joint
-    name="index1_index2" type="revolute">
+    name="${prefix}index1_index2" type="revolute">
     <origin xyz="0.001 -0.040 0.000" rpy="0 0 0" />
-    <parent link="index1" />
-    <child link="index2" />
-    <axis xyz="1 0 0" />
-    <limit lower="-0.697" upper="1.57" effort="10000" velocity="0.5"/>
-    <dynamics damping="5" friction="0.0"/>
-</joint>
-<link name="index2">
-    <inertial>
-      <origin xyz="0 0 0" rpy="0 0 0" />
-      <mass value="0.7" />
-          <inertia ixx="0.003" ixy="0" ixz="0" iyy="0.0030" iyz="0" izz="0.0035"/>
-    </inertial>
-    <visual>
-      <origin xyz="0 0 0" rpy="0 0 0" />
-      <geometry>
-        <mesh  filename="package://human_arm_description/meshes/index2.stl" />
-      </geometry>
-      <material name="">
-        <color rgba="0.79216 0.81961 0.93333 1" />
-      </material>
-    </visual>
-    <collision>
-      <origin xyz="0 0 0" rpy="0 0 0" />
-      <geometry>
-          <mesh  filename="package://human_arm_description/meshes/index2.stl" />
-      </geometry>
-    </collision>
-</link>
-<joint
-    name="index2_index3" type="revolute">
+    <parent link="${prefix}index1" />
+    <child link="${prefix}index2" />
+    <axis xyz="1 0 0" />
+    <limit lower="0" upper="1.57" effort="10000" velocity="0.5"/>
+    <dynamics damping="5" friction="0.0"/>
+</joint>
+<link name="${prefix}index2">
+    <inertial>
+      <origin xyz="0 0 0" rpy="0 0 0" />
+      <mass value="0.7" />
+          <inertia ixx="0.003" ixy="0" ixz="0" iyy="0.0030" iyz="0" izz="0.0035"/>
+    </inertial>
+    <visual>
+      <origin xyz="0 0 0" rpy="0 0 0" />
+      <geometry>
+        <mesh  filename="package://human_arm_description/meshes/index2.stl" scale="1 0.8 1" />
+      </geometry>
+      <material name="">
+        <color rgba="0.79216 0.81961 0.93333 1" />
+      </material>
+    </visual>
+    <collision>
+      <origin xyz="0 0 0" rpy="0 0 0" />
+      <geometry>
+          <mesh  filename="package://human_arm_description/meshes/index2.stl" scale="1 0.8 1" />
+      </geometry>
+    </collision>
+</link>
+<joint
+    name="${prefix}index2_index3" type="revolute">
     <origin xyz="0.00 -0.017 0.000" rpy="0 0 0" />
-    <parent link="index2" />
-    <child link="index3" />
-    <axis xyz="1 0 0" />
-    <limit lower="-0.697" upper="1.57" effort="10000" velocity="0.5"/>
-    <dynamics damping="5" friction="0.0"/>
-</joint>
-<link name="index3">
+    <parent link="${prefix}index2" />
+    <child link="${prefix}index3" />
+    <axis xyz="1 0 0" />
+    <limit lower="0" upper="1.57" effort="10000" velocity="0.5"/>
+    <dynamics damping="5" friction="0.0"/>
+</joint>
+<link name="${prefix}index3">
     <inertial>
       <origin xyz="0 0 0" rpy="0 0 0" />
@@ -371,13 +372,13 @@
 ##################### MIDDLE FINGER ######################################## -->
 <joint
-    name="palm_middle0" type="revolute">
+    name="${prefix}palm_middle0" type="revolute">
     <origin xyz="-0.011 -0.07 0.000" rpy="0 0 0" />
-    <parent link="palm" />
-    <child link="middle0" />
-    <axis xyz="0 0 1" />
-    <limit lower="-0.697" upper="1.57" effort="10000" velocity="0.5"/>
-    <dynamics damping="5" friction="0.0"/>
-</joint>
-<link name="middle0">
+    <parent link="${prefix}palm" />
+    <child link="${prefix}middle0" />
+    <axis xyz="0 0 1" />
+    <limit lower="-0.3" upper="0.3" effort="10000" velocity="0.5"/>
+    <dynamics damping="5" friction="0.0"/>
+</joint>
+<link name="${prefix}middle0">
     <inertial>
       <origin xyz="0 0 0" rpy="0 0 0" />
@@ -402,13 +403,13 @@
 </link>
 <joint
-    name="middle0_middle1" type="revolute">
+    name="${prefix}middle0_middle1" type="revolute">
     <origin xyz="0.00 -0.020 0.000" rpy="0 0 0" />
-    <parent link="middle0" />
-    <child link="middle1" />
-    <axis xyz="1 0 0" />
-    <limit lower="-0.697" upper="1.57" effort="10000" velocity="0.5"/>
-    <dynamics damping="5" friction="0.0"/>
-</joint>
-<link name="middle1">
+    <parent link="${prefix}middle0" />
+    <child link="${prefix}middle1" />
+    <axis xyz="1 0 0" />
+    <limit lower="-0.2" upper="1.57" effort="10000" velocity="0.5"/>
+    <dynamics damping="5" friction="0.0"/>
+</joint>
+<link name="${prefix}middle1">
     <inertial>
       <origin xyz="0 0 0" rpy="0 0 0" />
@@ -433,44 +434,44 @@
 </link>
 <joint
-    name="middle1_middle2" type="revolute">
+    name="${prefix}middle1_middle2" type="revolute">
     <origin xyz="0.001 -0.045 0.000" rpy="0 0 0" />
-    <parent link="middle1" />
-    <child link="middle2" />
-    <axis xyz="1 0 0" />
-    <limit lower="-0.697" upper="1.57" effort="10000" velocity="0.5"/>
-    <dynamics damping="5" friction="0.0"/>
-</joint>
-<link name="middle2">
-    <inertial>
-      <origin xyz="0 0 0" rpy="0 0 0" />
-      <mass value="0.7" />
-          <inertia ixx="0.003" ixy="0" ixz="0" iyy="0.0030" iyz="0" izz="0.0035"/>
-    </inertial>
-    <visual>
-      <origin xyz="0 0 0" rpy="0 0 0" />
-      <geometry>
-        <mesh  filename="package://human_arm_description/meshes/middle2.stl" />
-      </geometry>
-      <material name="">
-        <color rgba="0.79216 0.81961 0.93333 1" />
-      </material>
-    </visual>
-    <collision>
-      <origin xyz="0 0 0" rpy="0 0 0" />
-      <geometry>
-          <mesh  filename="package://human_arm_description/meshes/middle2.stl" />
-      </geometry>
-    </collision>
-</link>
-<joint
-    name="middle2_middle3" type="revolute">
+    <parent link="${prefix}middle1" />
+    <child link="${prefix}middle2" />
+    <axis xyz="1 0 0" />
+    <limit lower="0" upper="1.57" effort="10000" velocity="0.5"/>
+    <dynamics damping="5" friction="0.0"/>
+</joint>
+<link name="${prefix}middle2">
+    <inertial>
+      <origin xyz="0 0 0" rpy="0 0 0" />
+      <mass value="0.7" />
+          <inertia ixx="0.003" ixy="0" ixz="0" iyy="0.0030" iyz="0" izz="0.0035"/>
+    </inertial>
+    <visual>
+      <origin xyz="0 0 0" rpy="0 0 0" />
+      <geometry>
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