Commit message: gazebo bug fixed

File: human_arm_description/urdf/right_arm.xacro (robot description, xacro)
@@ -2,5 +2,5 @@
 <robot name="right_arm" xmlns:xacro="http://www.ros.org/wiki/xacro">
 <xacro:include filename="$(find human_arm_description)/urdf/right_arm.gazebo" />
-<xacro:property name="prefix" value="right_"/>
+<!-- <xacro:property name="prefix" value="right_"/> -->
 <link name="${prefix}shoulder">
     <inertial>
@@ -31,6 +31,6 @@
     <child link="${prefix}humerus" />
     <axis xyz="1 0 0" />
-    <limit lower="-3.14" upper="0.345" effort="10000" velocity="0.5"/>
-    <dynamics damping="5" friction="0.0"/>
+    <limit lower="-3.14" upper="0.345" effort="150.0" velocity="1"/>
+    <!-- dynamics damping="5" friction="0.0"/ -->
 </joint>
 <link name="${prefix}humerus">
@@ -62,6 +62,6 @@
     <child link="${prefix}elbow" />
     <axis xyz="0 1 0" />
-    <limit lower="-3.142" upper="0" effort="10000" velocity="0.5"/>
-    <dynamics damping="5" friction="0.0"/>
+    <limit lower="-3.142" upper="0" effort="150.0" velocity="1"/>
+    <!-- dynamics damping="5" friction="0.0"/ -->
 </joint>
 <link name="${prefix}elbow">
@@ -93,6 +93,6 @@
     <child link="${prefix}forearm" />
     <axis xyz="0 0 1" />
-    <limit lower="0" upper="2.4" effort="10000" velocity="0.5"/>
-    <dynamics damping="5" friction="0.0"/>
+    <limit lower="0" upper="2.4" effort="150.0" velocity="1"/>
+    <!-- dynamics damping="5" friction="0.0"/ -->
 </joint>
 <link name="${prefix}forearm">
@@ -124,6 +124,6 @@
     <child link="${prefix}wristy" />
     <axis xyz="0 1 0" />
-    <limit lower="-3.142" upper="2" effort="10000" velocity="0.5"/>
-    <dynamics damping="5" friction="0.0"/>
+    <limit lower="-3.142" upper="2" effort="150.0" velocity="1"/>
+    <!-- dynamics damping="5" friction="0.0"/ -->
 </joint>
 <link name="${prefix}wristy">
@@ -155,6 +155,6 @@
     <child link="${prefix}wristx" />
     <axis xyz="0 0 1" />
-    <limit lower="-0.697" upper="0.697" effort="10000" velocity="0.5"/>
-    <dynamics damping="5" friction="0.0"/>
+    <limit lower="-0.697" upper="0.697" effort="150.0" velocity="1"/>
+    <!-- dynamics damping="5" friction="0.0"/ -->
 </joint>
 <link name="${prefix}wristx">
@@ -186,6 +186,6 @@
     <child link="${prefix}wristz" />
     <axis xyz="1 0 0" />
-    <limit lower="-1" upper="1.57" effort="10000" velocity="0.5"/>
-    <dynamics damping="5" friction="0.0"/>
+    <limit lower="-1" upper="1.57" effort="150.0" velocity="1"/>
+    <!-- dynamics damping="5" friction="0.0"/ -->
 </joint>
 <link name="${prefix}wristz">
@@ -217,6 +217,6 @@
     <child link="${prefix}palm" />
     <axis xyz="0 0 1" />
-    <limit lower="-0.697" upper="1.57" effort="10000" velocity="0.5"/>
-    <dynamics damping="5" friction="0.0"/>
+    <limit lower="-0.697" upper="1.57" effort="150.0" velocity="1"/>
+    <!-- dynamics damping="5" friction="0.0"/ -->
 </joint>
 <link name="${prefix}palm">
@@ -251,6 +251,6 @@
     <child link="${prefix}index0" />
     <axis xyz="0 0 1" />
-    <limit lower="-0.3" upper="0.3" effort="10000" velocity="0.5"/>
-    <dynamics damping="5" friction="0.0"/>
+    <limit lower="-0.3" upper="0.3" effort="150.0" velocity="1"/>
+    <!-- dynamics damping="5" friction="0.0"/ -->
 </joint>
 <link name="${prefix}index0">
@@ -282,6 +282,6 @@
     <child link="${prefix}index1" />
     <axis xyz="1 0 0" />
-    <limit lower="-0.2" upper="1.57" effort="10000" velocity="0.5"/>
-    <dynamics damping="5" friction="0.0"/>
+    <limit lower="-0.2" upper="1.57" effort="150.0" velocity="1"/>
+    <!-- dynamics damping="5" friction="0.0"/ -->
 </joint>
 <link name="${prefix}index1">
@@ -313,6 +313,6 @@
     <child link="${prefix}index2" />
     <axis xyz="1 0 0" />
-    <limit lower="0" upper="1.57" effort="10000" velocity="0.5"/>
-    <dynamics damping="5" friction="0.0"/>
+    <limit lower="0" upper="1.57" effort="150.0" velocity="1"/>
+    <!-- dynamics damping="5" friction="0.0"/ -->
 </joint>
 <link name="${prefix}index2">
@@ -344,6 +344,6 @@
     <child link="${prefix}index3" />
     <axis xyz="1 0 0" />
-    <limit lower="0" upper="1.57" effort="10000" velocity="0.5"/>
-    <dynamics damping="5" friction="0.0"/>
+    <limit lower="0" upper="1.57" effort="150.0" velocity="1"/>
+    <!-- dynamics damping="5" friction="0.0"/ -->
 </joint>
 <link name="${prefix}index3">
@@ -378,6 +378,6 @@
     <child link="${prefix}middle0" />
     <axis xyz="0 0 1" />
-    <limit lower="-0.3" upper="0.3" effort="10000" velocity="0.5"/>
-    <dynamics damping="5" friction="0.0"/>
+    <limit lower="-0.3" upper="0.3" effort="150.0" velocity="1"/>
+    <!-- dynamics damping="5" friction="0.0"/ -->
 </joint>
 <link name="${prefix}middle0">
@@ -409,6 +409,6 @@
     <child link="${prefix}middle1" />
     <axis xyz="1 0 0" />
-    <limit lower="-0.2" upper="1.57" effort="10000" velocity="0.5"/>
-    <dynamics damping="5" friction="0.0"/>
+    <limit lower="-0.2" upper="1.57" effort="150.0" velocity="1"/>
+    <!-- dynamics damping="5" friction="0.0"/ -->
 </joint>
 <link name="${prefix}middle1">
@@ -440,6 +440,6 @@
     <child link="${prefix}middle2" />
     <axis xyz="1 0 0" />
-    <limit lower="0" upper="1.57" effort="10000" velocity="0.5"/>
-    <dynamics damping="5" friction="0.0"/>
+    <limit lower="0" upper="1.57" effort="150.0" velocity="1"/>
+    <!-- dynamics damping="5" friction="0.0"/ -->
 </joint>
 <link name="${prefix}middle2">
@@ -471,6 +471,6 @@
     <child link="${prefix}middle3" />
     <axis xyz="1 0 0" />
-    <limit lower="0" upper="1.57" effort="10000" velocity="0.5"/>
-    <dynamics damping="5" friction="0.0"/>
+    <limit lower="0" upper="1.57" effort="150.0" velocity="1"/>
+    <!-- dynamics damping="5" friction="0.0"/ -->
 </joint>
 <link name="${prefix}middle3">
@@ -505,6 +505,6 @@
     <child link="${prefix}ring0" />
     <axis xyz="0 0 1" />
-    <limit lower="-0.3" upper="0.3" effort="10000" velocity="0.5"/>
-    <dynamics damping="5" friction="0.0"/>
+    <limit lower="-0.3" upper="0.3" effort="150.0" velocity="1"/>
+    <!-- dynamics damping="5" friction="0.0"/ -->
 </joint>
 <link name="${prefix}ring0">
@@ -536,6 +536,6 @@
     <child link="${prefix}ring1" />
     <axis xyz="1 0 0" />
-    <limit lower="-0.2" upper="1.57" effort="10000" velocity="0.5"/>
-    <dynamics damping="5" friction="0.0"/>
+    <limit lower="-0.2" upper="1.57" effort="150.0" velocity="1"/>
+    <!-- dynamics damping="5" friction="0.0"/ -->
 </joint>
 <link name="${prefix}ring1">
@@ -567,6 +567,6 @@
     <child link="${prefix}ring2" />
     <axis xyz="1 0 0" />
-    <limit lower="0" upper="1.57" effort="10000" velocity="0.5"/>
-    <dynamics damping="5" friction="0.0"/>
+    <limit lower="0" upper="1.57" effort="150.0" velocity="1"/>
+    <!-- dynamics damping="5" friction="0.0"/ -->
 </joint>
 <link name="${prefix}ring2">
@@ -598,6 +598,6 @@
     <child link="${prefix}ring3" />
     <axis xyz="1 0 0" />
-    <limit lower="0" upper="1.57" effort="10000" velocity="0.5"/>
-    <dynamics damping="5" friction="0.0"/>
+    <limit lower="0" upper="1.57" effort="150.0" velocity="1"/>
+    <!-- dynamics damping="5" friction="0.0"/ -->
 </joint>
 <link name="${prefix}ring3">
@@ -632,6 +632,6 @@
     <child link="${prefix}pinky0" />
     <axis xyz="0 0 1" />
-    <limit lower="-0.3" upper="0.3" effort="10000" velocity="0.5"/>
-    <dynamics damping="5" friction="0.0"/>
+    <limit lower="-0.3" upper="0.3" effort="150.0" velocity="1"/>
+    <!-- dynamics damping="5" friction="0.0"/ -->
 </joint>
 <link name="${prefix}pinky0">
@@ -663,6 +663,6 @@
     <child link="${prefix}pinky1" />
     <axis xyz="1 0 0" />
-    <limit lower="-0.2" upper="1.57" effort="10000" velocity="0.5"/>
-    <dynamics damping="5" friction="0.0"/>
+    <limit lower="-0.2" upper="1.57" effort="150.0" velocity="1"/>
+    <!-- dynamics damping="5" friction="0.0"/ -->
 </joint>
 <link name="${prefix}pinky1">
@@ -694,6 +694,6 @@
     <child link="${prefix}pinky2" />
     <axis xyz="1 0 0" />
-    <limit lower="0" upper="1.57" effort="10000" velocity="0.5"/>
-    <dynamics damping="5" friction="0.0"/>
+    <limit lower="0" upper="1.57" effort="150.0" velocity="1"/>
+    <!-- dynamics damping="5" friction="0.0"/ -->
 </joint>
 <link name="${prefix}pinky2">
@@ -725,6 +725,6 @@
     <child link="${prefix}pinky3" />
     <axis xyz="1 0 0" />
-    <limit lower="0" upper="1.57" effort="10000" velocity="0.5"/>
-    <dynamics damping="5" friction="0.0"/>
+    <limit lower="0" upper="1.57" effort="150.0" velocity="1"/>
+    <!-- dynamics damping="5" friction="0.0"/ -->
 </joint>
 <link name="${prefix}pinky3">
@@ -755,12 +755,33 @@
 <joint
     name="${prefix}palm_thumb_zero" type="revolute">
-    <origin xyz="0.00 -0.02 0.000" rpy="0 0 0" />
+    <origin xyz="-0.005 -0.02 0.000" rpy="0 0 0" />
     <parent link="${prefix}palm" />
     <child link="${prefix}thumb_zero_zero" />
     <axis xyz="1 0 0" />
-    <limit lower="0" upper="1.8" effort="10000" velocity="0.5"/>
-    <dynamics damping="5" friction="0.0"/>
-</joint>
-<link name="${prefix}thumb_zero_zero"/>
+    <limit lower="0" upper="1.8" effort="150.0" velocity="1"/>
+    <!-- dynamics damping="5" friction="0.0"/ -->
+</joint>
+<link name="${prefix}thumb_zero_zero">
+    <inertial>
+      <origin xyz="0 0 0" rpy="0 0 0" />
+      <mass value="0.7" />
+          <inertia ixx="0.003" ixy="0" ixz="0" iyy="0.0030" iyz="0" izz="0.0035"/>
+    </inertial>
+    <visual>
+      <origin xyz="0 0 0" rpy="0 0 0" />
+      <geometry>
+        <cylinder length="0.005" radius="0.01"/>
+      </geometry>
+      <material name="">
+        <color rgba="0.79216 0.81961 0.93333 1" />
+      </material>
+    </visual>
+    <collision>
+      <origin xyz="0 0 0" rpy="0 0 0" />
+      <geometry>
+         <cylinder length="0.005" radius="0.01"/>
+      </geometry>
+    </collision>
+</link>
 <joint
     name="${prefix}palm_thumb0" type="revolute">
@@ -769,6 +790,6 @@
     <child link="${prefix}thumb0" />
     <axis xyz="0 1 0" />
-    <limit lower="0" upper="1.8" effort="10000" velocity="0.5"/>
-    <dynamics damping="5" friction="0.0"/>
+    <limit lower="0" upper="1.8" effort="150.0" velocity="1"/>
+    <!-- dynamics damping="5" friction="0.0"/ -->
 </joint>
 <link name="${prefix}thumb0">
@@ -800,6 +821,6 @@
     <child link="${prefix}thumb1" />
     <axis xyz="0 0 1" />
-    <limit lower="-1" upper="0" effort="10000" velocity="0.5"/>
-    <dynamics damping="5" friction="0.0"/>
+    <limit lower="-1" upper="0" effort="150.0" velocity="1"/>
+    <!-- dynamics damping="5" friction="0.0"/ -->
 </joint>
 <link name="${prefix}thumb1">
@@ -831,6 +852,6 @@
     <child link="${prefix}thumb2" />
     <axis xyz="0 0 1" />
-    <limit lower="-0.8" upper="0" effort="10000" velocity="0.5"/>
-    <dynamics damping="5" friction="0.0"/>
+    <limit lower="-0.8" upper="0" effort="150.0" velocity="1"/>
+    <!-- dynamics damping="5" friction="0.0"/ -->
 </joint>
 <link name="${prefix}thumb2">
@@ -862,6 +883,6 @@
     <child link="${prefix}thumb3" />
     <axis xyz="0 0 1" />
-    <limit lower="-0.697" upper="0" effort="10000" velocity="0.5"/>
-    <dynamics damping="5" friction="0.0"/>
+    <limit lower="-0.697" upper="0" effort="150.0" velocity="1"/>
+    <!-- dynamics damping="5" friction="0.0"/ -->
 </joint>
 <link name="${prefix}thumb3">

Commit message: Scaling factor changed in python api

File: human_arm_description/urdf/right_arm.xacro (robot description, xacro)
@@ -31,5 +31,5 @@
     <child link="${prefix}humerus" />
     <axis xyz="1 0 0" />
-    <limit lower="-3.14" upper="0.345" effort="150.0" velocity="1"/>
+    <limit lower="-3.14" upper="0.345" effort="150.0" velocity="3"/>
     <!-- dynamics damping="5" friction="0.0"/ -->
 </joint>
@@ -62,5 +62,5 @@
     <child link="${prefix}elbow" />
     <axis xyz="0 1 0" />
-    <limit lower="-3.142" upper="0" effort="150.0" velocity="1"/>
+    <limit lower="-3.142" upper="0" effort="150.0" velocity="3"/>
     <!-- dynamics damping="5" friction="0.0"/ -->
 </joint>
@@ -93,5 +93,5 @@
     <child link="${prefix}forearm" />
     <axis xyz="0 0 1" />
-    <limit lower="0" upper="2.4" effort="150.0" velocity="1"/>
+    <limit lower="0" upper="2.4" effort="150.0" velocity="3"/>
     <!-- dynamics damping="5" friction="0.0"/ -->
 </joint>
@@ -124,5 +124,5 @@
     <child link="${prefix}wristy" />
     <axis xyz="0 1 0" />
-    <limit lower="-3.142" upper="2" effort="150.0" velocity="1"/>
+    <limit lower="-3.142" upper="2" effort="150.0" velocity="3"/>
     <!-- dynamics damping="5" friction="0.0"/ -->
 </joint>
@@ -155,5 +155,5 @@
     <child link="${prefix}wristx" />
     <axis xyz="0 0 1" />
-    <limit lower="-0.697" upper="0.697" effort="150.0" velocity="1"/>
+    <limit lower="-0.697" upper="0.697" effort="150.0" velocity="3"/>
     <!-- dynamics damping="5" friction="0.0"/ -->
 </joint>
@@ -186,5 +186,5 @@
     <child link="${prefix}wristz" />
     <axis xyz="1 0 0" />
-    <limit lower="-1" upper="1.57" effort="150.0" velocity="1"/>
+    <limit lower="-1" upper="1.57" effort="150.0" velocity="3"/>
     <!-- dynamics damping="5" friction="0.0"/ -->
 </joint>
@@ -217,5 +217,5 @@
     <child link="${prefix}palm" />
     <axis xyz="0 0 1" />
-    <limit lower="-0.697" upper="1.57" effort="150.0" velocity="1"/>
+    <limit lower="-0.697" upper="1.57" effort="150.0" velocity="3"/>
     <!-- dynamics damping="5" friction="0.0"/ -->
 </joint>
@@ -251,5 +251,5 @@
     <child link="${prefix}index0" />
     <axis xyz="0 0 1" />
-    <limit lower="-0.3" upper="0.3" effort="150.0" velocity="1"/>
+    <limit lower="-0.3" upper="0.3" effort="150.0" velocity="3"/>
     <!-- dynamics damping="5" friction="0.0"/ -->
 </joint>
@@ -282,5 +282,5 @@
     <child link="${prefix}index1" />
     <axis xyz="1 0 0" />
-    <limit lower="-0.2" upper="1.57" effort="150.0" velocity="1"/>
+    <limit lower="-0.2" upper="1.57" effort="150.0" velocity="3"/>
     <!-- dynamics damping="5" friction="0.0"/ -->
 </joint>
@@ -313,5 +313,5 @@
     <child link="${prefix}index2" />
     <axis xyz="1 0 0" />
-    <limit lower="0" upper="1.57" effort="150.0" velocity="1"/>
+    <limit lower="0" upper="1.57" effort="150.0" velocity="3"/>
     <!-- dynamics damping="5" friction="0.0"/ -->
 </joint>
@@ -344,5 +344,5 @@
     <child link="${prefix}index3" />
     <axis xyz="1 0 0" />
-    <limit lower="0" upper="1.57" effort="150.0" velocity="1"/>
+    <limit lower="0" upper="1.57" effort="150.0" velocity="3"/>
     <!-- dynamics damping="5" friction="0.0"/ -->
 </joint>
@@ -378,5 +378,5 @@
     <child link="${prefix}middle0" />
     <axis xyz="0 0 1" />
-    <limit lower="-0.3" upper="0.3" effort="150.0" velocity="1"/>
+    <limit lower="-0.3" upper="0.3" effort="150.0" velocity="3"/>
     <!-- dynamics damping="5" friction="0.0"/ -->
 </joint>
@@ -409,5 +409,5 @@
     <child link="${prefix}middle1" />
     <axis xyz="1 0 0" />
-    <limit lower="-0.2" upper="1.57" effort="150.0" velocity="1"/>
+    <limit lower="-0.2" upper="1.57" effort="150.0" velocity="3"/>
     <!-- dynamics damping="5" friction="0.0"/ -->
 </joint>
@@ -440,5 +440,5 @@
     <child link="${prefix}middle2" />
     <axis xyz="1 0 0" />
-    <limit lower="0" upper="1.57" effort="150.0" velocity="1"/>
+    <limit lower="0" upper="1.57" effort="150.0" velocity="3"/>
     <!-- dynamics damping="5" friction="0.0"/ -->
 </joint>
@@ -471,5 +471,5 @@
     <child link="${prefix}middle3" />
     <axis xyz="1 0 0" />
-    <limit lower="0" upper="1.57" effort="150.0" velocity="1"/>
+    <limit lower="0" upper="1.57" effort="150.0" velocity="3"/>
     <!-- dynamics damping="5" friction="0.0"/ -->
 </joint>
@@ -505,5 +505,5 @@
     <child link="${prefix}ring0" />
     <axis xyz="0 0 1" />
-    <limit lower="-0.3" upper="0.3" effort="150.0" velocity="1"/>
+    <limit lower="-0.3" upper="0.3" effort="150.0" velocity="3"/>
     <!-- dynamics damping="5" friction="0.0"/ -->
 </joint>
@@ -536,5 +536,5 @@
     <child link="${prefix}ring1" />
     <axis xyz="1 0 0" />
-    <limit lower="-0.2" upper="1.57" effort="150.0" velocity="1"/>
+    <limit lower="-0.2" upper="1.57" effort="150.0" velocity="3"/>
     <!-- dynamics damping="5" friction="0.0"/ -->
 </joint>
@@ -567,5 +567,5 @@
     <child link="${prefix}ring2" />
     <axis xyz="1 0 0" />
-    <limit lower="0" upper="1.57" effort="150.0" velocity="1"/>
+    <limit lower="0" upper="1.57" effort="150.0" velocity="3"/>
     <!-- dynamics damping="5" friction="0.0"/ -->
 </joint>
@@ -598,5 +598,5 @@
     <child link="${prefix}ring3" />
     <axis xyz="1 0 0" />
-    <limit lower="0" upper="1.57" effort="150.0" velocity="1"/>
+    <limit lower="0" upper="1.57" effort="150.0" velocity="3"/>
     <!-- dynamics damping="5" friction="0.0"/ -->
 </joint>
@@ -632,5 +632,5 @@
     <child link="${prefix}pinky0" />
     <axis xyz="0 0 1" />
-    <limit lower="-0.3" upper="0.3" effort="150.0" velocity="1"/>
+    <limit lower="-0.3" upper="0.3" effort="150.0" velocity="3"/>
     <!-- dynamics damping="5" friction="0.0"/ -->
 </joint>
@@ -663,5 +663,5 @@
     <child link="${prefix}pinky1" />
     <axis xyz="1 0 0" />
-    <limit lower="-0.2" upper="1.57" effort="150.0" velocity="1"/>
+    <limit lower="-0.2" upper="1.57" effort="150.0" velocity="3"/>
     <!-- dynamics damping="5" friction="0.0"/ -->
 </joint>
@@ -694,5 +694,5 @@
     <child link="${prefix}pinky2" />
     <axis xyz="1 0 0" />
-    <limit lower="0" upper="1.57" effort="150.0" velocity="1"/>
+    <limit lower="0" upper="1.57" effort="150.0" velocity="3"/>
     <!-- dynamics damping="5" friction="0.0"/ -->
 </joint>
@@ -725,5 +725,5 @@
     <child link="${prefix}pinky3" />
     <axis xyz="1 0 0" />
-    <limit lower="0" upper="1.57" effort="150.0" velocity="1"/>
+    <limit lower="0" upper="1.57" effort="150.0" velocity="3"/>
     <!-- dynamics damping="5" friction="0.0"/ -->
 </joint>
@@ -759,5 +759,5 @@
     <child link="${prefix}thumb_zero_zero" />
     <axis xyz="1 0 0" />
-    <limit lower="0" upper="1.8" effort="150.0" velocity="1"/>
+    <limit lower="0" upper="1.8" effort="150.0" velocity="3"/>
     <!-- dynamics damping="5" friction="0.0"/ -->
 </joint>
@@ -790,5 +790,5 @@
     <child link="${prefix}thumb0" />
     <axis xyz="0 1 0" />
-    <limit lower="0" upper="1.8" effort="150.0" velocity="1"/>
+    <limit lower="0" upper="1.8" effort="150.0" velocity="3"/>
     <!-- dynamics damping="5" friction="0.0"/ -->
 </joint>
@@ -821,5 +821,5 @@
     <child link="${prefix}thumb1" />
     <axis xyz="0 0 1" />
-    <limit lower="-1" upper="0" effort="150.0" velocity="1"/>
+    <limit lower="-1" upper="0" effort="150.0" velocity="3"/>
     <!-- dynamics damping="5" friction="0.0"/ -->
 </joint>
@@ -852,5 +852,5 @@
     <child link="${prefix}thumb2" />
     <axis xyz="0 0 1" />
-    <limit lower="-0.8" upper="0" effort="150.0" velocity="1"/>
+    <limit lower="-0.8" upper="0" effort="150.0" velocity="3"/>
     <!-- dynamics damping="5" friction="0.0"/ -->
 </joint>
@@ -883,5 +883,5 @@
     <child link="${prefix}thumb3" />
     <axis xyz="0 0 1" />
-    <limit lower="-0.697" upper="0" effort="150.0" velocity="1"/>
+    <limit lower="-0.697" upper="0" effort="150.0" velocity="3"/>
     <!-- dynamics damping="5" friction="0.0"/ -->
 </joint>
